Commit message: ankle limit

File: software/resources/robots/asimov_v1/urdf/asimov_v1_legs.urdf (robot description, URDF)
Before this commit: robot asimov_v1_legs, 28 links, 27 joints
Joints:
- joint left_ankle_pitch_joint: limit lower=-0.35 upper=0.35 effort=200 velocity=20 -> lower=-0.7 upper=0.7 effort=200 velocity=20
- joint left_ankle_roll_joint: limit lower=-0.1 upper=0.1 effort=200 velocity=20 -> lower=-0.3 upper=0.3 effort=200 velocity=20
- joint right_ankle_pitch_joint: limit lower=-0.35 upper=0.35 effort=200 velocity=20 -> lower=-0.7 upper=0.7 effort=200 velocity=20
- joint right_ankle_roll_joint: limit lower=-0.1 upper=0.1 effort=200 velocity=20 -> lower=-0.3 upper=0.3 effort=200 velocity=20

Commit message: ankle

File: software/resources/robots/asimov_v1/urdf/asimov_v1_legs.urdf (robot description, URDF)
Before this commit: robot asimov_v1_legs, 28 links, 27 joints
Joints:
- joint left_ankle_pitch_joint: limit lower=-0.7 upper=0.7 effort=200 velocity=20 -> lower=-0.35 upper=0.35 effort=200 velocity=20
- joint left_ankle_roll_joint: limit lower=-0.3 upper=0.3 effort=200 velocity=20 -> lower=-0.1 upper=0.1 effort=200 velocity=20
- joint right_ankle_pitch_joint: limit lower=-0.7 upper=0.7 effort=200 velocity=20 -> lower=-0.35 upper=0.35 effort=200 velocity=20
- joint right_ankle_roll_joint: limit lower=-0.3 upper=0.3 effort=200 velocity=20 -> lower=-0.1 upper=0.1 effort=200 velocity=20
