Commit message: fix: ankle limit collision, ankle_roll range, restore mirror_mask
Three regressions introduced in eb7d1ad (ankle) and 534f195 (lin_vel_x):

1. ankle swing delta ±0.13 → ±0.08
   default ±0.25 + delta ±0.13 = ±0.38 exceeded the ±0.35 URDF hard
   limit, so the ankle hit the physical stop on every swing cycle and
   the PD controller saturated. Peak is now ±0.33, 2° inside the soft
   limit (0.98×0.35=0.343).

2. ankle_roll limit ±0.10 → ±0.20 (URDF + MJCF)
   eb7d1ad reduced ankle_roll from ±0.30 to ±0.10 (5.7°), leaving
   almost no lateral correction authority during single-leg stance.
   ±0.20 restores enough range for balance without exceeding hardware.

3. Restore mirror_mask in asimov_stand_env.py and sim2sim.py
   534f195 removed the mask added in 943e872 to fix asymmetric gait
   (v28: only left leg lifts). Without it the policy sees raw URDF
   sign-flipped right-side joints and converges to asymmetric local
   optima. mask: [1]*6 + [-1]*6 applied on obs path, un-applied on
   action path and in sim2sim.py inference.

Co-Authored-By: Claude Sonnet 4.6 (1M context) <noreply@anthropic.com>

File: software/resources/robots/asimov_v1/urdf/asimov_v1_legs.urdf (robot description, URDF)
Before this commit: robot asimov_v1_legs, 28 links, 27 joints
Joints:
- joint left_ankle_roll_joint: limit lower=-0.1 upper=0.1 effort=200 velocity=20 -> lower=-0.2 upper=0.2 effort=200 velocity=20
- joint right_ankle_roll_joint: limit lower=-0.1 upper=0.1 effort=200 velocity=20 -> lower=-0.2 upper=0.2 effort=200 velocity=20
